File: PCB/SAMPad.kicad_pcb (KiCad board)
At the start: 2 copper layers, 73.2 x 116 mm, 155 parts, among them P1 USB_CONN, P1_2 USB_CONN, P4 CONN_6, P5 CONN_6, P6 ISP6, U1 ATMEGA32U4, U3 IP4234CZ6, U5 PAM2804, X1 CRYSTAL

Commit message: Rev 0.6
Parts:
- removed R9: 100k, prettylib:SMD_0805
- JP1: footprint prettylib:JUMPER_SMD_2 -> prettylib:JUMPER_SMD_3
- R1: value 1k -> 10k
- moved R35 6.82 mm to (149.6, 84.5), turned to 90 degrees
- moved C23 3.53 mm to (151.8, 84.5), turned to 270 degrees
- moved C22 3.34 mm to (162.4, 84.5), turned to 270 degrees
- moved R34 2.57 mm to (159.2, 86.5)
- moved R1 1.59 mm to (101.5, 148.7), turned to 0 degrees
- moved LOGO1 1.12 mm to (128.1, 86.0)
- moved LOGO2 1.12 mm to (129.1, 86.0)
- moved JP1 0.89 mm to (96.6, 148.4)
Connections:
- JP1 pad 1: Net-(JP1-Pad1) -> +5V
- JP1 pad 2: /mcu/HWBE -> VSS
- R1 pad 2: Net-(JP1-Pad1) -> /mcu/HWBE
Routing:
- net VSS: track 462.9 -> 486.2 mm
- net +5V: track 518.6 -> 526.7 mm
- net /mcu/HWBE: track 27.9 -> 20.3 mm
- net /mcu/ENCB: track 86.0 -> 91.3 mm
- net Net-(JP1-Pad1): track 2.78 -> 0.00 mm
- net /ledmatrix/LEDI6: track 97.3 -> 98.5 mm
- net /mcu/ENCA: track 97.6 -> 96.4 mm
Other:
- outline, holes or cut-outs redrawn
- board text added: "SAMPad Rev 0.6 Designed & Drawin in KiCAD by Mohit 'MOZ' Garg"
- board text added: "SAMPad Rev 0.6 Designed & Drawn in KiCAD by Mohit 'MOZ' Garg"
- board text removed: "SAMPad Rev 0.5 Designed & Drawin in KiCAD by Mohit 'MOZ' Garg Use EasyAVR to Program"
- board text removed: "SAMPad Rev 0.5 Designed & Drawn in KiCAD by Mohit 'MOZ' Garg Use EasyAVR to Program"
